File: 2-Schematic/kicad.kicad_pcb (KiCad board)
At the start: 2 copper layers, 9 parts, among them J1 MYCONN3, U1 PIC12C508A-ISN

Commit message: fix issue
Parts:
- removed the D1 at (149.9, 104.1)
- removed the R2 at (101.6, 110.5)
- removed R3: R, Resistor_THT:R_Axial_DIN0207_L6.3mm_D2.5mm_P15.24mm_Horizontal
- removed the U1 at (87.5, 37.1)
- moved J1 50.9 mm to (131.3, 76.1)
Connections:
- R2 pad 1: /INPUT -> (no net)
- U1 pad 2: Net-(U1-Pad2) -> (no net)
- U1 pad 3: Net-(U1-Pad3) -> (no net)
- U1 pad 4: Net-(U1-Pad4) -> (no net)
- U1 pad 5: Net-(U1-Pad5) -> (no net)
- U1 pad 6: Net-(U1-Pad6) -> (no net)
