File: 3-Bus/kicad/kicad.sch (KiCad schematic (older format))
At the start: 0 parts

Commit message: update bus.sch
Parts:
- added P10: CONN_1, symbol Connector_Generic:Conn_01x04
- added P11: CONN_2, symbol Connector_Generic:Conn_01x04
- added P12: CONN_3, symbol Connector_Generic:Conn_01x04
- added P13: CONN_4, symbol Connector_Generic:Conn_01x04
Changed lines of the file:
@@
 Comment4 ""
 $EndDescr
+$Comp
+L Connector_Generic:Conn_01x04 P10
+U 1 1 5DEF6D3E
+P 2950 2400
+F 0 "P10" H 2868 2717 50  0000 C CNN
+F 1 "CONN_1" H 2868 2626 50  0000 C CNN
+F 2 "" H 2950 2400 50  0001 C CNN
+F 3 "~" H 2950 2400 50  0001 C CNN
+	1    2950 2400
+	-1   0    0    -1
+$EndComp
+$Comp
+L Connector_Generic:Conn_01x04 P11
+U 1 1 5DEF7733
+P 2950 3150
+F 0 "P11" H 2868 3467 50  0000 C CNN
+F 1 "CONN_2" H 2868 3376 50  0000 C CNN
+F 2 "" H 2950 3150 50  0001 C CNN
+F 3 "~" H 2950 3150 50  0001 C CNN
+	1    2950 3150
+	-1   0    0    -1
+$EndComp
+$Comp
+L Connector_Generic:Conn_01x04 P12
+U 1 1 5DEF814B
+P 2950 3900
+F 0 "P12" H 2868 4217 50  0000 C CNN
+F 1 "CONN_3" H 2868 4126 50  0000 C CNN
+F 2 "" H 2950 3900 50  0001 C CNN
+F 3 "~" H 2950 3900 50  0001 C CNN
+	1    2950 3900
+	-1   0    0    -1
+$EndComp
+Entry Wire Line
+	3600 3050 3500 3150
+Entry Wire Line
+	3600 2950 3500 3050
+Entry Wire Line
+	3600 3250 3500 3350
+Entry Wire Line
+	3600 3150 3500 3250
+Entry Wire Line
+	3600 3800 3500 3900
+Entry Wire Line
+	3500 3800 3600 3700
+Entry Wire Line
+	3500 4000 3600 3900
+Entry Wire Line
+	3500 4100 3600 4000
+Entry Wire Line
+	3600 2500 3500 2600
+Entry Wire Line
+	3500 2500 3600 2400
+Entry Wire Line
+	3500 2400 3600 2300
+Entry Wire Line
+	3600 2200 3500 2300
+$Comp
+L Connector_Generic:Conn_01x04 P13
+U 1 1 5DEF8B8E
+P 5100 2400
+F 0 "P13" H 5180 2392 50  0000 L CNN
+F 1 "CONN_4" H 5180 2301 50  0000 L CNN
+F 2 "" H 5100 2400 50  0001 C CNN
+F 3 "~" H 5100 2400 50  0001 C CNN
+	1    5100 2400
+	1    0    0    -1
+$EndComp
+Entry Wire Line
+	4500 2200 4600 2300
+Entry Wire Line
+	4500 2300 4600 2400
+Entry Wire Line
+	4500 2400 4600 2500
+Entry Wire Line
+	4500 2500 4600 2600
 $EndSCHEMATC
