File: 4-PCB/kicad.kicad_pcb (KiCad board)
At the start: 2 copper layers, 5 parts, among them J1 MYCONN3, U1 PIC12C508A-ISN

Commit message: PCB layout
Parts:
- moved R1 3.58 mm to (131.7, 101.3), turned to 180 degrees
- moved D1 1.99 mm to (131.7, 89.4)
- moved R2 1.76 mm to (159.6, 89.2)
- moved U1 1.76 mm to (141.9, 94.2)
- moved J1 1.76 mm to (129.4, 114.6)
Routing:
- net GND: track 0.00 -> 50.8 mm, vias 0 -> 1
- net /INPUTtoR: track 0.00 -> 34.1 mm
- net VCC: track 0.00 -> 28.5 mm
- net /INPUT: track 0.00 -> 15.2 mm
- net Net-(D1-Pad1): track 0.00 -> 14.8 mm
- net /LEDtoR: track 0.00 -> 11.9 mm
- added copper zone on B.Cu, net GND
Other:
- board outline added: 44.5 x 38.4 mm
