File: Tutorial/uinio.kicad_pcb (KiCad board)
At the start: 2 copper layers, 64 x 39 mm, 3 parts

Commit message: update
Parts:
- added SW1: M2011S3A1W03, Getting_Started:Switch_Toggle_SPST_NKK_M2011S3A1x03, F.Cu at (163.5, 77.0)
Connections:
- BT1 pad 1: VCC -> unconnected-(BT1-Pad1)
- R1 pad 2: VCC -> unconnected-(R1-Pad2)
Routing:
- net unconnected-(BT1-Pad1): track 0.00 -> 28.1 mm
- net VCC: track 28.1 -> 0.00 mm
Changed lines of the file:
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@@
   (net 2 "GND")
   (net 3 "/LED")
+  (net 4 "unconnected-(BT1-Pad1)")
+  (net 5 "unconnected-(R1-Pad2)")
+  (net 6 "unconnected-(SW1-Pad2)")
+  (footprint "Getting_Started:Switch_Toggle_SPST_NKK_M2011S3A1x03" (layer "F.Cu")
+    (at 163.46 76.96)
+    (property "Sheetfile" "uinio.kicad_sch")
+    (property "Sheetname" "")
+    (attr through_hole)
+    (fp_text reference "SW1" (at -1.94 -2.91 unlocked) (layer "F.SilkS")
+      (effects (font (size 1 1) (thickness 0.15)))
+    )
+    (fp_text value "M2011S3A1W03" (at 0.06 13.09 unlocked) (layer "F.Fab")
+      (effects (font (size 1 1) (thickness 0.15)))
+    )
+    (fp_text user "${REFERENCE}" (at 0 2.5 unlocked) (layer "F.Fab")
+      (effects (font (size 1 1) (thickness 0.15)))
+    )
+    (fp_rect (start -4.06 -1.91) (end 4.06 11.31) (layer "F.SilkS") (width 0.12) (fill none))
+    (fp_rect (start -4.2 -2.05) (end 4.2 11.45) (layer "F.CrtYd") (width 0.05) (fill none))
+    (fp_rect (start -3.95 -1.8) (end 3.95 11.2) (layer "F.Fab") (width 0.1) (fill none))
+    (pad "2" thru_hole circle (at 0 4.7) (size 2.22 2.22) (drill 1.62) (layers *.Cu *.Mask)
+      (net 6 "unconnected-(SW1-Pad2)") (pinfunction "A") (pintype "passive"))
+    (pad "3" thru_hole circle (at 0 9.4) (size 2.22 2.22) (drill 1.62) (layers *.Cu *.Mask)
+      (net 1 "VCC") (pinfunction "B") (pintype "passive"))
+  )
   (footprint "LED_THT:LED_D5.0mm" (layer "F.Cu")
     (at 178.5 74.225 -90)
@@
       (net 3 "/LED") (pintype "passive"))
     (pad "2" thru_hole oval (at 12.7 0 180) (size 1.6 1.6) (drill 0.8) (layers *.Cu *.Mask)
-      (net 1 "VCC") (pintype "passive"))
+      (net 5 "unconnected-(R1-Pad2)") (pintype "passive"))
     (model "${KICAD6_3DMODEL_DIR}/Resistor_THT.3dshapes/R_Axial_DIN0309_L9.0mm_D3.2mm_P12.70mm_Horizontal.wrl"
       (offset (xyz 0 0 0))
@@
     (fp_arc (start -10.61275 -3.5) (mid -9.478596 -5.91918) (end -7.802602 -7.999992) (layer "B.Fab") (width 0.1))
     (pad "1" smd rect (at -14.68 0 90) (size 2.54 3.51) (layers "B.Cu" "B.Paste" "B.Mask")
-      (net 1 "VCC") (pinfunction "+") (pintype "passive"))
+      (net 4 "unconnected-(BT1-Pad1)") (pinfunction "+") (pintype "passive"))
     (pad "2" smd rect (at 14.68 0 90) (size 2.54 3.51) (layers "B.Cu" "B.Paste" "B.Mask")
       (net 2 "GND") (pinfunction "-") (pintype "passive"))
@@
   )
   (gr_rect (start 131 60.5) (end 195 99.5) (layer "Edge.Cuts") (width 0.1) (fill none))
-  (segment (start 148.3 95.2) (end 165.8 95.2) (width 0.25) (layer "B.Cu") (net 1))
-  (segment (start 147 95.18) (end 148.28 95.18) (width 0.25) (layer "B.Cu") (net 1))
-  (segment (start 172.15 88.85) (end 172.15 88.5) (width 0.25) (layer "B.Cu") (net 1))
-  (segment (start 148.28 95.18) (end 148.3 95.2) (width 0.25) (layer "B.Cu") (net 1))
-  (segment (start 165.8 95.2) (end 172.15 88.85) (width 0.25) (layer "B.Cu") (net 1))
   (segment (start 170.95 74.2) (end 168.45 74.2) (width 0.25) (layer "F.Cu") (net 2))
   (segment (start 160.15 65.9) (end 157.5 65.9) (width 0.25) (layer "F.Cu") (net 2))
@@
   (segment (start 184.85 88.5) (end 184.85 83.115) (width 0.25) (layer "B.Cu") (net 3))
   (segment (start 184.85 83.115) (end 178.5 76.765) (width 0.25) (layer "B.Cu") (net 3))
+  (segment (start 148.3 95.2) (end 165.8 95.2) (width 0.25) (layer "B.Cu") (net 4))
+  (segment (start 147 95.18) (end 148.28 95.18) (width 0.25) (layer "B.Cu") (net 4))
+  (segment (start 172.15 88.85) (end 172.15 88.5) (width 0.25) (layer "B.Cu") (net 4))
+  (segment (start 148.28 95.18) (end 148.3 95.2) (width 0.25) (layer "B.Cu") (net 4))
+  (segment (start 165.8 95.2) (end 172.15 88.85) (width 0.25) (layer "B.Cu") (net 4))
   (zone (net 2) (net_name "GND") (layer "B.Cu") (hatch edge 0.508)
     (connect_pads (clearance 0.508))

Commit message: finish all of job
Parts:
- moved D1 20.1 mm to (168.0, 91.4), turned to 0 degrees
- moved SW1 12.7 mm to (173.6, 69.3), turned to 90 degrees
- moved R1 3.46 mm to (183.0, 91.4), turned to 90 degrees
- turned BT1 to -90 degrees
Connections:
- net /LED renamed Net-(D1-Pad2)
- BT1 pad 1: unconnected-(BT1-Pad1) -> Net-(BT1-Pad1)
- R1 pad 2: unconnected-(R1-Pad2) -> VCC
- SW1 pad 2: unconnected-(SW1-Pad2) -> Net-(BT1-Pad1)
Routing:
- net Net-(BT1-Pad1): track 0.00 -> 32.8 mm
- net unconnected-(BT1-Pad1): track 28.1 -> 0.00 mm
- net GND: track 35.0 -> 23.9 mm, vias 2 -> 0
- net VCC: track 0.00 -> 9.90 mm
- net Net-(D1-Pad2): track 14.4 -> 12.5 mm
Other:
- board text added: "UinIO.com by Hank"
